File: buck.brd (EAGLE design)
At the start: 100 x 100 mm, 252 parts, among them J1 SSM-105-XXX-DV, J2 SSM-105-XXX-DV, J3 SSM-105-XXX-DV, Q1 BSS123, Q10 BSS123, Q11 BSS123, Q12 BSS123, Q13 BSS123, Q14 BSS123, Q15 BSS123, Q16 BSS123, Q2 BSS123, Q5 BSS123, Q6 BSS123, Q7 BSS123, Q8 BSS123, Q9 BSS123, U2 TPS54531DDA_3D, U3 TPS54531DDA_3D, U4 TPS54531DDA_3D, U5 TPS54531DDA_3D, U6 TPS54531DDA_3D, U7 TPS54531DDA_3D, U8 TPS54531DDA_3D

Commit message: final version v1.0
Parts:
- added C10, C4, C5, C6, C7, C8, C9: 100n, rcl:C0603K
- moved C46 0.32 mm to (35.7, 56.2)
- moved R53 0.32 mm to (30.8, 36.4)
- moved C108 0.16 mm to (68.1, 18.1)
- moved C33 0.16 mm to (68.1, 54.9)
- moved C93 0.16 mm to (68.1, 74.0)
- moved C106 0.16 mm to (63.7, 27.6)
- moved C61 0.16 mm to (36.4, 37.1)
- moved LED4 0.16 mm to (47.8, 66.0)
- moved R51 0.16 mm to (37.9, 37.1)
- moved LED5 0.16 mm to (20.2, 19.4)
- moved C14 0.16 mm to (40.8, 65.7)
- moved C48 0.16 mm to (40.8, 46.7)
- moved C63 0.16 mm to (40.8, 27.6)
- moved C78 0.16 mm to (40.8, 8.57)
- moved LED2 0.16 mm to (20.5, 57.5)
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Connections:
- removed net N$10: U$5.2
- removed net N$8: U$5.6
- removed net N$88: U$5.3
- removed net N$89: U$5.1
- removed net N$9: U$5.4
- new net CANH2: U$1.2, U$2.1
- new net CANL2: U$1.4, U$2.3
- new net WDO_5V1: C5.1, R12.1, R13.2, U2.3
- net GND: now also C10.2, C4.2, C5.2, C6.2, C7.2, C8.2, C9.2, U$5.1, U$5.2, U$5.3, U$5.4, U$5.6; no longer U$1.2, U$1.4, U$2.1, U$2.3
- net WDO_13V: now also C10.1
- net WDO_3V8: no longer R12.1, R13.2, U2.3
- net WDO_3V8': now also C8.1
- net WDO_5V5: now also C4.1
- net WDO_5V5': now also C7.1
- net WDO_6V6: now also C6.1
- net WDO_7V4: now also C9.1
Routing:
- net GND: track 117.8 -> 96.7 mm, vias 373 -> 378
- net SUPPLY1: track 13.5 -> 0.00 mm, vias 2 -> 5
- net WDO_5V1: track 0.00 -> 11.6 mm, vias 0 -> 1
- net WDO_3V8: track 52.6 -> 41.7 mm
- net RECO_5: track 5.72 -> 0.00 mm, vias 1 -> 2
- net LINE3: track 4.32 -> 0.00 mm, vias 1 -> 2
- net LINE2: track 4.32 -> 0.00 mm, vias 1 -> 2
- net CANL2: track 0.00 -> 4.32 mm, vias 0 -> 1
- net CANH2: track 0.00 -> 4.32 mm, vias 0 -> 1
- net PWM2: track 4.32 -> 0.00 mm, vias 1 -> 2
- net PWM1: track 4.32 -> 0.00 mm, vias 1 -> 2
- net LINE7: track 4.32 -> 0.00 mm, vias 1 -> 2
- net LINE6: track 4.32 -> 0.00 mm, vias 1 -> 2
- net POWER1: track 4.34 -> 0.04 mm, vias 0 -> 2
- net POWER2: track 4.21 -> 0.00 mm, vias 1 -> 2
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- added copper zone on layer 1, net LINE2
- added copper zone on layer 16, net LINE2
- added copper zone on layer 1, net LINE3
- added copper zone on layer 16, net LINE3
- added copper zone on layer 1, net LINE6
- added copper zone on layer 16, net LINE6
- added copper zone on layer 1, net LINE7
- added copper zone on layer 16, net LINE7
- added copper zone on layer 1, net POWER1
- added copper zone on layer 16, net POWER1
- added copper zone on layer 1, net POWER2
- added copper zone on layer 16, net POWER2
- added copper zone on layer 1, net PWM1
- added copper zone on layer 16, net PWM1
- added copper zone on layer 1, net PWM2
- added copper zone on layer 16, net PWM2
- added copper zone on layer 1, net RECO_5
- added copper zone on layer 16, net RECO_5
- added copper zone on layer 1, net SUPPLY1
- added copper zone on layer 16, net SUPPLY1
Other:
- board text added: "Bucks Converter"
- board text added: "Tomasz Tatara"

Commit message: version 2 for production
Parts:
- removed J1, J2: SSM-105-XXX-DV, SMD_254_10:SSM-105-XXX-DV
- added U$13, U$14: IPT1-110-01-X-D-VS, smd_2.54_20pos:IPT1-110-01-X-D-VS
Connections:
- net LINE6 renamed STASZEK_OUT2
- net LINE7 renamed STASZEK_OUT1
- net POWER1 renamed RECO_POWER1
- net POWER2 renamed RECO_POWER2
- net PWM1 renamed RECO_POWER3
- net PWM2 renamed RECO_POWER4
- net RECO_5 renamed SERVO_RECO2
- net R_SPI_MISO renamed STASZEK_SERVO1
- net R_SPI_MOSI renamed STASZEK_SERVO2
- net R_SPI_SCK renamed FREE1
- net SUPPLY1 renamed SYSTEM_SUPPLY
- net WATCHDOG renamed CAN2H
- removed net ANALOG1+: J1.1, J2.2
- removed net ANALOG1-: J1.3, J2.4
- removed net ANALOG2+: J1.5, J2.6
- removed net ANALOG2-: J1.7, J2.8
- removed net ANALOG3+: J1.8, J2.7
- removed net ANALOG3-: J1.10, J2.9
- removed net CANH2: U$1.2, U$2.1
- removed net CANL2: U$1.4, U$2.3
- removed net ENGINE_BURNOUT1: J1.4, J2.3
- removed net ENGINE_BURNOUT2: J1.2, J2.1
- removed net GNDA: J1.9, J2.10
- removed net LINE1: J1.6, J2.5
- removed net LINE2: U$3.9, U$4.10
- removed net LINE3: U$3.7, U$4.8
- new net +11: U$13.14, U$14.13
- new net AGND: U$13.6, U$14.5
- new net BURNOUT+: U$13.10, U$14.9
- new net BURNOUT-: U$13.8, U$14.7
- new net CAN2L: U$3.16, U$4.15
- new net FREE2: U$3.6, U$4.5
- new net MAGNETO_SCL: U$13.18, U$14.17
- new net MAGNETO_SDA: U$13.16, U$14.15
- new net MAGNETO_SUPPLY: U$13.20, U$14.19
- new net PITOT_CONN: U$13.17, U$14.18
- new net PITOT_OUT: U$13.15, U$14.16
- new net PITOT_SUPPLY: U$13.19, U$14.20
- new net PRESS1: U$13.12, U$14.11
- new net PRESS2: U$13.13, U$14.14
- new net PRESS3: U$13.11, U$14.12
- new net SERVO_RX: U$13.3, U$14.4
- new net SERVO_TX: U$13.1, U$14.2
- new net STASZEK_OUT3: U$1.7, U$2.8
- new net STASZEK_OUT4: U$1.13, U$2.14
- new net STASZEK_RECO_PWM: U$3.8, U$4.7
- new net STASZEK_SERVO3: U$13.2, U$14.1
- new net STASZEK_SERVO4: U$13.4, U$14.3
- new net TEMP1: U$13.9, U$14.10
- new net TEMP2: U$13.7, U$14.8
- new net TEMP3: U$13.5, U$14.6
- net 13V: no longer U$1.16, U$2.15
- net 3V8: no longer U$3.6, U$4.5
- net 3V8': now also U$1.6, U$2.5; no longer U$1.7, U$2.8
- net 5V5: now also U$3.9, U$4.10; no longer U$3.8, U$4.7
- net 5V5': now also U$1.16, U$2.15; no longer U$1.13, U$2.14
- net 6V6: now also U$3.13, U$4.14; no longer U$3.16, U$4.15
- net GND: now also U$1.2, U$1.4, U$2.1, U$2.3; no longer U$1.6, U$2.5
- net SERVO_RECO1: now also U$3.7, U$4.8; no longer U$3.13, U$4.14
Routing:
- net 3V8: track 34.1 -> 18.6 mm, vias 15 -> 11
- net 13V: track 36.2 -> 23.2 mm, vias 17 -> 13
- net 7V4: track 40.8 -> 32.1 mm, vias 19 -> 17
- net 6V6: track 34.7 -> 26.1 mm, vias 14 -> 16
- net 3V8': track 37.7 -> 29.1 mm, vias 13 -> 14
- net 5V5: track 39.3 -> 30.7 mm, vias 14 -> 16
- net 5V5': track 35.5 -> 26.8 mm, vias 8 -> 12
- net GND: track 96.7 -> 91.9 mm, vias 378 -> 366
- net STASZEK_SERVO2: track 4.32 -> 0.00 mm, vias 1 -> 2
- net STASZEK_SERVO1: track 4.32 -> 0.00 mm, vias 1 -> 2
- net SERVO_RECO1: track 4.32 -> 0.00 mm, vias 1 -> 2
- net FREE1: track 4.32 -> 0.00 mm, vias 1 -> 2
- net CANL2: track 4.32 -> 0.00 mm, vias 1 -> 0
- net CANH2: track 4.32 -> 0.00 mm, vias 1 -> 0
- net CAN2H: track 4.32 -> 0.00 mm, vias 1 -> 2
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- added copper zone on layer 1, net +11
- added copper zone on layer 16, net +11
- added copper zone on layer 1, net AGND
- added copper zone on layer 16, net AGND
- added copper zone on layer 1, net BURNOUT+
- added copper zone on layer 16, net BURNOUT+
- added copper zone on layer 1, net BURNOUT-
- added copper zone on layer 16, net BURNOUT-
- added copper zone on layer 1, net CAN2H
- added copper zone on layer 16, net CAN2H
- added copper zone on layer 1, net CAN2L
- added copper zone on layer 16, net CAN2L
- added copper zone on layer 1, net CANH
- added copper zone on layer 16, net CANH
- added copper zone on layer 1, net CANL
- added copper zone on layer 16, net CANL
- added copper zone on layer 1, net FREE1
- added copper zone on layer 16, net FREE1
- added copper zone on layer 1, net FREE2
- added copper zone on layer 16, net FREE2
- added copper zone on layer 1, net MAGNETO_SCL
- added copper zone on layer 16, net MAGNETO_SCL
- added copper zone on layer 1, net MAGNETO_SDA
- added copper zone on layer 16, net MAGNETO_SDA
- added copper zone on layer 1, net MAGNETO_SUPPLY
- added copper zone on layer 16, net MAGNETO_SUPPLY
- added copper zone on layer 1, net PITOT_CONN
- added copper zone on layer 16, net PITOT_CONN
- added copper zone on layer 1, net PITOT_OUT
- added copper zone on layer 16, net PITOT_OUT
- added copper zone on layer 1, net PITOT_SUPPLY
- added copper zone on layer 16, net PITOT_SUPPLY
- added copper zone on layer 1, net PRESS1
- added copper zone on layer 16, net PRESS1
- added copper zone on layer 1, net PRESS2
- added copper zone on layer 16, net PRESS2
- added copper zone on layer 1, net PRESS3
- added copper zone on layer 16, net PRESS3
- added copper zone on layer 1, net SERVO_RECO1
- added copper zone on layer 16, net SERVO_RECO1
- added copper zone on layer 1, net SERVO_RX
- added copper zone on layer 16, net SERVO_RX
- added copper zone on layer 1, net SERVO_TX
- added copper zone on layer 16, net SERVO_TX
- added copper zone on layer 1, net STASZEK_OUT3
- added copper zone on layer 16, net STASZEK_OUT3
- added copper zone on layer 1, net STASZEK_OUT4
- added copper zone on layer 16, net STASZEK_OUT4
- added copper zone on layer 1, net STASZEK_RECO_PWM
- added copper zone on layer 16, net STASZEK_RECO_PWM
- added copper zone on layer 1, net STASZEK_SERVO1
- added copper zone on layer 16, net STASZEK_SERVO1
- added copper zone on layer 1, net STASZEK_SERVO2
- added copper zone on layer 16, net STASZEK_SERVO2
- added copper zone on layer 1, net STASZEK_SERVO3
- added copper zone on layer 16, net STASZEK_SERVO3
- added copper zone on layer 1, net STASZEK_SERVO4
- added copper zone on layer 16, net STASZEK_SERVO4
- added copper zone on layer 1, net TEMP1
- added copper zone on layer 16, net TEMP1
- added copper zone on layer 1, net TEMP2
- added copper zone on layer 16, net TEMP2
- added copper zone on layer 1, net TEMP3
- added copper zone on layer 16, net TEMP3
- removed copper zone on layer 1, net LINE2
- removed copper zone on layer 16, net LINE2
- removed copper zone on layer 1, net LINE3
- removed copper zone on layer 16, net LINE3
