File: buck.sch (EAGLE design)
At the start: 252 parts, among them J1 SSM-105-XXX-DV, J2 SSM-105-XXX-DV, J3 SSM-105-XXX-DV, Q1 BSS123, Q10 BSS123, Q11 BSS123, Q12 BSS123, Q13 BSS123, Q14 BSS123, Q15 BSS123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

Commit message: final version v1.0
Parts:
- added C10, C4, C5, C6, C7, C8, C9: 100n, rcl:C-EUC0603K
Connections:
- removed net N$10: U$5.2
- removed net N$8: U$5.6
- removed net N$88: U$5.3
- removed net N$89: U$5.1
- removed net N$9: U$5.4
- new net CANH2: U$1.2, U$2.1
- new net CANL2: U$1.4, U$2.3
- new net WDO_5V1: C5.1, R12.1, R13.2, U2.EN
- net GND: now also C10.2, C4.2, C5.2, C6.2, C7.2, C8.2, C9.2, U$5.1, U$5.2, U$5.3, U$5.4, U$5.6; no longer U$1.2, U$1.4, U$2.1, U$2.3
- net WDO_13V: now also C10.1
- net WDO_3V8: no longer R12.1, R13.2, U2.EN
- net WDO_3V8': now also C8.1
- net WDO_5V5: now also C4.1
- net WDO_5V5': now also C7.1
- net WDO_6V6: now also C6.1
- net WDO_7V4: now also C9.1

Commit message: version 2 for production
Parts:
- removed J1, J2: SSM-105-XXX-DV, SMD_254_10:SSM-105-XXX-DV
- added U$13, U$14: IPT1-110-01-X-D-VS, smd_2.54_20pos:IPT1-110-01-X-D-VS
Connections:
- net LINE6 renamed STASZEK_OUT2
- net LINE7 renamed STASZEK_OUT1
- net POWER1 renamed RECO_POWER1
- net POWER2 renamed RECO_POWER2
- net PWM1 renamed RECO_POWER3
- net PWM2 renamed RECO_POWER4
- net RECO_5 renamed SERVO_RECO2
- net R_SPI_MISO renamed STASZEK_SERVO1
- net R_SPI_MOSI renamed STASZEK_SERVO2
- net R_SPI_SCK renamed FREE1
- net SUPPLY1 renamed SYSTEM_SUPPLY
- net WATCHDOG renamed CAN2H
- removed net ANALOG1+: J1.1, J2.2
- removed net ANALOG1-: J1.3, J2.4
- removed net ANALOG2+: J1.5, J2.6
- removed net ANALOG2-: J1.7, J2.8
- removed net ANALOG3+: J1.8, J2.7
- removed net ANALOG3-: J1.10, J2.9
- removed net CANH2: U$1.2, U$2.1
- removed net CANL2: U$1.4, U$2.3
- removed net ENGINE_BURNOUT1: J1.4, J2.3
- removed net ENGINE_BURNOUT2: J1.2, J2.1
- removed net GNDA: J1.9, J2.10
- removed net LINE1: J1.6, J2.5
- removed net LINE2: U$3.9, U$4.10
- removed net LINE3: U$3.7, U$4.8
- new net +11: U$13.14, U$14.13
- new net AGND: U$13.6, U$14.5
- new net BURNOUT+: U$13.10, U$14.9
- new net BURNOUT-: U$13.8, U$14.7
- new net CAN2L: U$3.16, U$4.15
- new net FREE2: U$3.6, U$4.5
- new net MAGNETO_SCL: U$13.18, U$14.17
- new net MAGNETO_SDA: U$13.16, U$14.15
- new net MAGNETO_SUPPLY: U$13.20, U$14.19
- new net PITOT_CONN: U$13.17, U$14.18
- new net PITOT_OUT: U$13.15, U$14.16
- new net PITOT_SUPPLY: U$13.19, U$14.20
- new net PRESS1: U$13.12, U$14.11
- new net PRESS2: U$13.13, U$14.14
- new net PRESS3: U$13.11, U$14.12
- new net SERVO_RX: U$13.3, U$14.4
- new net SERVO_TX: U$13.1, U$14.2
- new net STASZEK_OUT3: U$1.7, U$2.8
- new net STASZEK_OUT4: U$1.13, U$2.14
- new net STASZEK_RECO_PWM: U$3.8, U$4.7
- new net STASZEK_SERVO3: U$13.2, U$14.1
- new net STASZEK_SERVO4: U$13.4, U$14.3
- new net TEMP1: U$13.9, U$14.10
- new net TEMP2: U$13.7, U$14.8
- new net TEMP3: U$13.5, U$14.6
- net 13V: no longer U$1.16, U$2.15
- net 3V8: no longer U$3.6, U$4.5
- net 3V8': now also U$1.6, U$2.5; no longer U$1.7, U$2.8
- net 5V5: now also U$3.9, U$4.10; no longer U$3.8, U$4.7
- net 5V5': now also U$1.16, U$2.15; no longer U$1.13, U$2.14
- net 6V6: now also U$3.13, U$4.14; no longer U$3.16, U$4.15
- net GND: now also U$1.2, U$1.4, U$2.1, U$2.3; no longer U$1.6, U$2.5
- net SERVO_RECO1: now also U$3.7, U$4.8; no longer U$3.13, U$4.14
